Commit message: rotate the top camera

File: seat_car_description/urdf/include/sensors.xacro (robot description, xacro)
@@ -143,5 +143,5 @@
     <parent link="camera_board"/>
     <child link="top_camera"/>
-    <origin xyz="0.019 0 0.0405" rpy="0 -${PI/2} ${PI}"/>
+    <origin xyz="0.019 0 0.0405" rpy="0 ${PI/2} ${PI}"/>
   </joint>
   <link name="top_camera_optical">
